Commit message: Evo: make one canonical file the single source of physical truth
The same physical constant used to be declared in many places with mutually
incompatible values (four wheel diameters, three track widths). Introduce
bamboo_base/config/robots/bamboo4WD_V4_WSEsp32.yaml as the only place that
carries geometry, motorisation and PID gains, in native ROS parameter form so
it is directly usable by ros2 param load.

The driver becomes an authoritative consumer: esp32_driver.yaml keeps transport
and frames only, driver.launch.py loads the canonical file second (so it cannot
be contradicted), and the node declares every physical parameter WITHOUT a
default - a missing one now fails explicitly instead of silently falling back
to a placeholder.

The URDF reads the same source: wheel_radius and wheel_pos_y become xacro
arguments passed by description.launch.py, keeping the upstream values as
standalone defaults only.

Values are seeds, not measurements: every unmeasured line is marked so in the
file, and calibration remains lot 4.

Co-Authored-By: Claude Opus 5 <noreply@anthropic.com>

File: linorobot2_description/urdf/4wd_properties.urdf.xacro (robot description, xacro)
@@ -5,8 +5,15 @@
   <xacro:property name="base_height" value="0.129" />
   <xacro:property name="base_mass" value="10" />
-  <xacro:property name="wheel_radius" value="0.07162" />
+  <!-- Geometrie de roue : ARGUMENTS, pas des constantes. La verite physique vit dans
+       bamboo_base/config/robots/<robot>.yaml et est passee par description.launch.py
+       (wheel_radius = wheel_diameter_m / 2, wheel_pos_y = wheel_separation_m / 2).
+       Les defauts ci-dessous sont les valeurs de l'amont linorobot2 : ce ne sont PAS des
+       mesures de ce robot, elles ne servent qu'a garder le xacro utilisable seul. -->
+  <xacro:arg name="wheel_radius" default="0.07162" />
+  <xacro:arg name="wheel_pos_y" default="0.1355" />
+  <xacro:property name="wheel_radius" value="$(arg wheel_radius)" />
   <xacro:property name="wheel_width" value="0.05" />
   <xacro:property name="wheel_pos_x" value="0.120" />
-  <xacro:property name="wheel_pos_y" value="0.1355" />
+  <xacro:property name="wheel_pos_y" value="$(arg wheel_pos_y)" />
   <xacro:property name="wheel_pos_z" value="-0.04788" />
   <xacro:property name="wheel_mass" value=".6" />

Commit message: Evo: seed the canonical geometry with the WaveShare vendor figures
The single source of physical truth carried unmeasured placeholders. Replace
them with the constants WaveShare ships for this very kit (UGV Rover,
mainType 02) in its own firmware for the same General Driver board:
waveshareteam/ugv_base_general -> General_Driver/ugv_config.h.

  counts_per_rev      2114 -> 1650   (ONE_CIRCLE_PLUSES)
  wheel_separation_m  0.30 -> 0.172  (TRACK_WIDTH)
  wheel_diameter_m    0.08 confirmed (WHEEL_D)

The pulse count transfers as is because the counting is identical on both
sides: same encoder pins (M1 35/34, M2 16/27) and same attachHalfQuad mode.
Their ROS description (waveshareteam/ugv_ws, ros2-humble-develop) confirms
the figures independently, so the chassis xacro now takes its body, wheel
and axle dimensions from that URDF and its meshes instead of upstream
linorobot2 values that described a robot twice as long.

Also fix the two motor voltages, which were swapped with respect to
config/custom/bamboov310_config.h and quartered the RPM ceiling (106
instead of 425).

The vendor PID gains are deliberately NOT copied: their controller
regulates m/s with a 255 anti-windup, a different formulation from ours.
These are vendor values, not measurements of this robot; the lot 4
calibration still has to confirm them.

Co-Authored-By: Claude Opus 5 <noreply@anthropic.com>

File: linorobot2_description/urdf/4wd_properties.urdf.xacro (robot description, xacro)
@@ -1,22 +1,36 @@
 <?xml version="1.0"?>
 <robot xmlns:xacro="http://ros.org/wiki/xacro">
-  <xacro:property name="base_length" value="0.445" />
-  <xacro:property name="base_width" value="0.200" />
-  <xacro:property name="base_height" value="0.129" />
-  <xacro:property name="base_mass" value="10" />
+  <!-- Chassis du robot BambooWS (kit WaveShare "UGV Rover", mainType 02).
+       Dimensions relevees sur la description constructeur : depot
+       waveshareteam/ugv_ws (branche ros2-humble-develop),
+       src/ugv_main/ugv_description/urdf/ugv_rover.urdf et ses maillages STL.
+       Le maillage de caisse mesure 0.2452 x 0.2304 x 0.1211 m (largeur mesuree
+       au plus large, garde-boue compris : c'est ce qu'il faut pour l'empreinte
+       Nav2). La boite etant centree sur base_link, on lui donne la hauteur
+       utile au-dessus de l'axe des roues plutot que la hauteur totale. -->
+  <xacro:property name="base_length" value="0.245" />
+  <xacro:property name="base_width" value="0.230" />
+  <xacro:property name="base_height" value="0.080" />
+  <xacro:property name="base_mass" value="2.78" />
   <!-- Geometrie de roue : ARGUMENTS, pas des constantes. La verite physique vit dans
        bamboo_base/config/robots/<robot>.yaml et est passee par description.launch.py
        (wheel_radius = wheel_diameter_m / 2, wheel_pos_y = wheel_separation_m / 2).
-       Les defauts ci-dessous sont les valeurs de l'amont linorobot2 : ce ne sont PAS des
-       mesures de ce robot, elles ne servent qu'a garder le xacro utilisable seul. -->
-  <xacro:arg name="wheel_radius" default="0.07162" />
-  <xacro:arg name="wheel_pos_y" default="0.1355" />
+       Les defauts ci-dessous sont les valeurs constructeur du meme kit, pour que le
+       xacro reste utilisable seul ; ce ne sont PAS des mesures de ce robot. -->
+  <xacro:arg name="wheel_radius" default="0.04" />
+  <xacro:arg name="wheel_pos_y" default="0.086" />
   <xacro:property name="wheel_radius" value="$(arg wheel_radius)" />
-  <xacro:property name="wheel_width" value="0.05" />
-  <xacro:property name="wheel_pos_x" value="0.120" />
+  <xacro:property name="wheel_width" value="0.0425" />
+  <!-- demi-empattement et hauteur d'axe, releves sur les joints du constructeur
+       (roues a x = +/-0.0855, z = -0.041212 sous base_link). -->
+  <xacro:property name="wheel_pos_x" value="0.0855" />
   <xacro:property name="wheel_pos_y" value="$(arg wheel_pos_y)" />
-  <xacro:property name="wheel_pos_z" value="-0.04788" />
-  <xacro:property name="wheel_mass" value=".6" />
+  <xacro:property name="wheel_pos_z" value="-0.041212" />
+  <xacro:property name="wheel_mass" value="0.21" />
   <xacro:property name="wheel_torque" value="20" />
+  <!-- Poses de capteurs heritees de l'amont linorobot2 : le lidar de BambooWS
+       n'est PAS encore choisi (phase navigation suivante) et il n'y a pas de
+       camera de profondeur. Ces deux poses sont donc des valeurs d'attente, a
+       reprendre au montage du capteur reel. -->
   <xacro:property name="laser_pose">
     <origin xyz="-0.0475 0 0.125" rpy="0 0 0"/>

Commit message: Evo: navigation groundwork: robot-declared sensors, lidar and navigation blocks, wiring
- The BambooWS canonical file declares its sensors (lidar d500, camera, imu, battery),
  the lidar (LD19 family, /dev/lidar, 230400, frame, scan direction, crop, range, pose)
  and the navigation facts (Nav2 params file, maps dir, cautious speed limits).
- layout.py: lidar, navigation and control (cmd_vel mux) become wirable groups with
  their logical flows and fallbacks; mismatched ends of scan and cmd_vel_nav are flagged.
  BambooWS layout.yaml wires them.
- The URDF laser pose comes from lidar.pose_* through new xacro arguments instead of
  the upstream placeholder.
- docker/fetch_sources.sh clones third-party sources at a pinned commit into the
  git-ignored third_party/ (ldlidar_stl_ros2, no Humble apt package); rosbuild.sh lists
  the new packages.

Co-Authored-By: Claude Opus 5.5 <noreply@anthropic.com>

File: linorobot2_description/urdf/4wd_properties.urdf.xacro (robot description, xacro)
@@ -33,6 +33,13 @@
        camera de profondeur. Ces deux poses sont donc des valeurs d'attente, a
        reprendre au montage du capteur reel. -->
+  <!-- Pose du LIDAR : arguments xacro, POUSSES par description.launch.py depuis le bloc
+       `lidar.pose_*` du fichier canonique du robot (lot NAV). Les defauts sont les valeurs
+       d'attente de l'amont. -->
+  <xacro:arg name="laser_x" default="-0.0475" />
+  <xacro:arg name="laser_y" default="0.0" />
+  <xacro:arg name="laser_z" default="0.125" />
+  <xacro:arg name="laser_yaw" default="0.0" />
   <xacro:property name="laser_pose">
-    <origin xyz="-0.0475 0 0.125" rpy="0 0 0"/>
+    <origin xyz="$(arg laser_x) $(arg laser_y) $(arg laser_z)" rpy="0 0 $(arg laser_yaw)"/>
   </xacro:property>
   <xacro:property name="depth_sensor_pose">
